File: ex00/cao/button.sch (KiCad schematic (older format))
At the start: 4 parts, among them SW2 SW_Push, U9 +5V

Commit message: [ADD] finish
Parts:
- renumbered GND13 to GND
Changed lines of the file:
@@
 $Descr A4 11693 8268
 encoding utf-8
-Sheet 7 8
+Sheet 8 8
 Title ""
 Date ""
@@
 $EndDescr
 $Comp
-L cao_comp:Ground GND13
+L cao_comp:Ground GND
 U 1 1 5FCF0352
 P 1350 1700
-AR Path="/5FC31A06/5FCF0352" Ref="GND13"  Part="1"
-AR Path="/5FC30220/5FCF0352" Ref="GND12"  Part="1"
-F 0 "GND12" H 1479 1708 50  0000 L CNN
+AR Path="/5FC31A06/5FCF0352" Ref="GND"  Part="1"
+AR Path="/5FC30220/5FCF0352" Ref="GND"  Part="1"
+F 0 "GND" H 1479 1708 50  0000 L CNN
 F 1 "Ground" H 1350 2050 50  0001 C CNN
 F 2 "" H 1350 1700 50  0001 C CNN
@@
 AR Path="/5FC31A06/5FCF06B0" Ref="U9"  Part="1"
 AR Path="/5FC30220/5FCF06B0" Ref="U8"  Part="1"
-F 0 "U8" H 1350 800 50  0001 C CNN
+F 0 "U9" H 1350 800 50  0001 C CNN
 F 1 "+5V" H 1402 855 50  0000 L CNN
 F 2 "" H 1350 800 50  0001 C CNN
@@
 AR Path="/5FC31A06/5FCF10CD" Ref="SW2"  Part="1"
 AR Path="/5FC30220/5FCF10CD" Ref="SW1"  Part="1"
-F 0 "SW1" V 1304 1519 50  0000 L CNN
+F 0 "SW2" V 1304 1519 50  0000 L CNN
 F 1 "SW_Push" V 1395 1519 50  0000 L CNN
 F 2 "" H 1450 1375 50  0001 C CNN
@@
 AR Path="/5FC31A06/5FCF176F" Ref="R6"  Part="1"
 AR Path="/5FC30220/5FCF176F" Ref="R5"  Part="1"
-F 0 "R5" V 1304 1091 50  0000 L CNN
+F 0 "R6" V 1304 1091 50  0000 L CNN
 F 1 "10K" V 1395 1091 50  0000 L CNN
 F 2 "" H 1350 1000 50  0001 C CNN
