File: ex00/cao/cao.sch (KiCad schematic (older format))
At the start: 5 parts

Commit message: [ADD] peut le faire avec un peu de chance
Parts:
- removed C?: Capacitor, symbol cao_comp:Capacitor
- removed D?: LED, symbol cao_comp:LED
- removed R?: Resistor, symbol cao_comp:Resistor
- removed Y? (x2): Quartz, symbol cao_comp:Quartz
- added C1, C2: 22pF, symbol cao_comp:Capacitor
- added C4: 100nF, symbol cao_comp:Capacitor
- added C5: 10uF, symbol cao_comp:Capacitor
- added GND1, GND2, GND3, GND4, GND5, GND6: Ground, symbol cao_comp:Ground
- added H1: MountingHole, symbol cao_comp:MountingHole
- added J2: AVR-ISP-6, symbol cao_comp:AVR-ISP-6
- added P1, P2: PWR_FLAG, symbol cao_comp:PWR_FLAG
- added U1: ATmega328P-AU, symbol cao_comp:ATmega328P-AU
- added U2, U3, U4, U5, U6: +5V, symbol cao_comp:+5V
- added Y1: Quartz, symbol cao_comp:Quartz
Connections:
- new net: U1.18 (AVCC), U1.4 (VCC), U3.~
- new net: U1.20 (AREF), U2.~
- new net: GND1.~, U1.3 (GND)
- new net: J2.2 (VCC), U6.~
- new net: GND5.~, J2.6 (GND)
- new net: GND3.~, Y1.2
- new net: C1.2, C2.2, GND4.~, Y1.4
- new net: C4.1, C5.1, U4.~
- new net: C4.2, C5.2, GND2.~
- new net: P1.1, U5.~
- new net: GND6.~, P2.1
- new net BUT_0: U1.1 (PD3)
- new net LED_0: U1.12 (PB0)
- new net LED_1: U1.13 (PB1)
- new net LED_2: U1.14 (PB2)
- new net LED_3: J2.4 (MOSI), U1.15 (PB3)
- new net MCU_RX: U1.31 (PD1)
- new net MCU_TX: U1.30 (PD0)
- new net MISO: J2.1 (MISO), U1.16 (PB4)
- new net RESET: J2.5 (~RST), U1.29 (~RESET~/PC6)
- new net SCK: J2.3 (SCK), U1.17 (PB5)
- new net XTAL1: C2.1, U1.7 (XTAL1/PB6), Y1.1
- new net XTAL2: C1.1, U1.8 (XTAL2/PB7), Y1.3
- no-connect marks 0 -> 13

Commit message: [ADD] finish
Parts:
- renumbered GND4 to GND, GND3 to GND, GND2 to GND, GND1 to GND, GND6 to GND, GND5 to GND
Changed lines of the file:
@@
 $EndComp
 $Comp
-L cao_comp:Ground GND4
+L cao_comp:Ground GND
 U 1 1 5FC352B4
 P 3800 3100
-F 0 "GND4" H 3929 3108 50  0000 L CNN
+F 0 "GND" H 3929 3108 50  0000 L CNN
 F 1 "Ground" H 3800 3450 50  0001 C CNN
 F 2 "" H 3800 3100 50  0001 C CNN
@@
 	3500 2000 4150 2000
 $Comp
-L cao_comp:Ground GND3
+L cao_comp:Ground GND
 U 1 1 5FC3ABA5
 P 3800 2150
-F 0 "GND3" H 3700 2100 50  0000 R CNN
+F 0 "GND" H 3700 2100 50  0000 R CNN
 F 1 "Ground" H 3800 2500 50  0001 C CNN
 F 2 "" H 3800 2150 50  0001 C CNN
@@
 $EndComp
 $Comp
-L cao_comp:Ground GND2
+L cao_comp:Ground GND
 U 1 1 5FC931C6
 P 3150 1400
-F 0 "GND2" H 3279 1408 50  0000 L CNN
+F 0 "GND" H 3279 1408 50  0000 L CNN
 F 1 "Ground" H 3150 1750 50  0001 C CNN
 F 2 "" H 3150 1400 50  0001 C CNN
@@
 	1500 1750 1750 1750
 $Comp
-L cao_comp:Ground GND1
+L cao_comp:Ground GND
 U 1 1 5FCAFCFA
 P 2150 4450
-F 0 "GND1" H 2279 4458 50  0000 L CNN
+F 0 "GND" H 2279 4458 50  0000 L CNN
 F 1 "Ground" H 2150 4800 50  0001 C CNN
 F 2 "" H 2150 4450 50  0001 C CNN
@@
 $EndComp
 $Comp
-L cao_comp:Ground GND6
+L cao_comp:Ground GND
 U 1 1 5FCB7A54
 P 7200 4450
-F 0 "GND6" H 7329 4458 50  0000 L CNN
+F 0 "GND" H 7329 4458 50  0000 L CNN
 F 1 "Ground" H 7200 4800 50  0001 C CNN
 F 2 "" H 7200 4450 50  0001 C CNN
@@
 $EndComp
 $Comp
-L cao_comp:Ground GND5
+L cao_comp:Ground GND
 U 1 1 5FCCE3F6
 P 6900 1500
-F 0 "GND5" H 7029 1508 50  0000 L CNN
+F 0 "GND" H 7029 1508 50  0000 L CNN
 F 1 "Ground" H 6900 1850 50  0001 C CNN
 F 2 "" H 6900 1500 50  0001 C CNN
@@
 U 1 1 5FD00E0B
 P 3500 2750
-F 0 "C1" V 3454 2895 50  0000 L CNN
-F 1 "22pF" V 3545 2895 50  0000 L CNN
+F 0 "C1" V 3450 2450 50  0000 L CNN
+F 1 "22pF" V 3550 2400 50  0000 L CNN
 F 2 "" H 3500 2950 50  0001 C CNN
 F 3 "" H 3500 2950 50  0001 C CNN
