File: ex00/cao/led.sch (KiCad schematic (older format))
At the start: 3 parts

Commit message: [ADD] finish
Parts:
- renumbered GND7 to GND
Changed lines of the file:
@@
 	3750 1700 3200 1700
 $Comp
-L cao_comp:Ground GND7
+L cao_comp:Ground GND
 U 1 1 5FBF119A
 P 1750 1950
-AR Path="/5FC03ED2/5FBF119A" Ref="GND7"  Part="1"
-AR Path="/5FC25D47/5FBF119A" Ref="GND8"  Part="1"
-AR Path="/5FC261EB/5FBF119A" Ref="GND9"  Part="1"
-AR Path="/5FC26691/5FBF119A" Ref="GND10"  Part="1"
-F 0 "GND7" H 1879 1958 50  0000 L CNN
+AR Path="/5FC03ED2/5FBF119A" Ref="GND"  Part="1"
+AR Path="/5FC25D47/5FBF119A" Ref="GND"  Part="1"
+AR Path="/5FC261EB/5FBF119A" Ref="GND"  Part="1"
+AR Path="/5FC26691/5FBF119A" Ref="GND"  Part="1"
+F 0 "GND" H 1879 1958 50  0000 L CNN
 F 1 "Ground" H 1750 2300 50  0001 C CNN
 F 2 "" H 1750 1950 50  0001 C CNN
