File: ex00/cao/usb_flasher.sch (KiCad schematic (older format))
At the start: 4 parts, among them J11 Conn_01x06, U7 +5V

Commit message: [ADD] finish
Parts:
- renumbered GND11 to GND
Changed lines of the file:
@@
 $EndComp
 $Comp
-L cao_comp:Ground GND11
+L cao_comp:Ground GND
 U 1 1 5FC2C347
 P 2150 1450
-F 0 "GND11" V 2150 1321 50  0000 R CNN
+F 0 "GND" V 2150 1321 50  0000 R CNN
 F 1 "Ground" H 2150 1800 50  0001 C CNN
 F 2 "" H 2150 1450 50  0001 C CNN
